File: Hardware/Kicad/Rele-Wifi/Rele-Wifi.kicad_pcb (KiCad board)
At the start: 2 copper layers, 59 x 61.5 mm, 20 parts, among them U1 817C, U2 817C

Commit message: Terminamos el esquematico
Parts:
- added C1: 0.33 uF, Capacitor_SMD:C_0805_2012Metric, F.Cu at (96.7, 114.5)
- added C2: 0.1 uF, Capacitor_SMD:C_0805_2012Metric, F.Cu at (81.5, 107.7)
- added D5: ~, EESTN5:Led_0805, F.Cu at (116.1, 103.4)
- added D6: ~, EESTN5:Led_0805, F.Cu at (116.1, 125.0)
- added D7: ~, Diode_SMD:D_0805_2012Metric, F.Cu at (129.4, 94.2)
- added D8: ~, Diode_SMD:D_0805_2012Metric, F.Cu at (129.3, 115.9)
- added J10: ~, TerminalBlock:TerminalBlock_Xinya_XY308-2.54-3P_1x03_P2.54mm_Horizontal, F.Cu at (159.2, 95.8)
- added J11: ~, TerminalBlock:TerminalBlock_Xinya_XY308-2.54-3P_1x03_P2.54mm_Horizontal, F.Cu at (159.2, 128.1)
- added J12: ~, TerminalBlock:TerminalBlock_Xinya_XY308-2.54-3P_1x03_P2.54mm_Horizontal, F.Cu at (159.2, 117.2)
- added J13: Screw_Terminal_01x02, TerminalBlock:TerminalBlock_bornier-2_P5.08mm, F.Cu at (96.7, 125.2)
- added J7: ~, EESTN5:Jumper, F.Cu at (121.4, 93.3)
- added J8: ~, EESTN5:Jumper, F.Cu at (121.4, 115.0)
- added J9: ~, TerminalBlock:TerminalBlock_Xinya_XY308-2.54-3P_1x03_P2.54mm_Horizontal, F.Cu at (159.2, 106.2)
- added K3: ~, Relay_THT:Relay_DPDT_Finder_30.22, F.Cu at (133.2, 102.8)
- added K4: ~, Relay_THT:Relay_DPDT_Finder_30.22, F.Cu at (133.1, 124.4)
- added Q3: ~, Package_TO_SOT_SMD:SOT-23, F.Cu at (128.4, 99.4)
- added Q4: ~, Package_TO_SOT_SMD:SOT-23, F.Cu at (128.4, 120.6)
- added R5: 1K, Resistor_SMD:R_0805_2012Metric_Pad1.20x1.40mm_HandSolder, F.Cu at (116.1, 93.3)
- added R6: 1K, Resistor_SMD:R_0805_2012Metric_Pad1.20x1.40mm_HandSolder, F.Cu at (116.0, 115.0)
- added R7: 510, Resistor_SMD:R_0805_2012Metric_Pad1.20x1.40mm_HandSolder, F.Cu at (129.4, 104.4)
- added R8: 510, Resistor_SMD:R_0805_2012Metric_Pad1.20x1.40mm_HandSolder, F.Cu at (129.3, 126.3)
- added U3: 817C, Package_DIP:DIP-4_W7.62mm, F.Cu at (115.1, 98.2)
- added U4: 817C, Package_DIP:DIP-4_W7.62mm, F.Cu at (115.0, 119.4)
- added U5: L7805, Package_TO_SOT_SMD:TO-263-3_TabPin2, F.Cu at (83.0, 123.1)
- added U7: ESP32_DevKit_V1_CH9102X, EESTN5:ESP32-WROOM-32.30pines, F.Cu at (93.8, 68.0)
- J2, J3, J4, J5: footprint TerminalBlock:TerminalBlock_MaiXu_MX126-5.0-03P_1x03_P5.00mm -> TerminalBlock:TerminalBlock_Xinya_XY308-2.54-3P_1x03_P2.54mm_Horizontal
- Q1, Q2: footprint Package_TO_SOT_THT:TO-126-3_Vertical -> Package_TO_SOT_SMD:SOT-23
- moved J1 26.8 mm to (121.8, 51.2)
- moved J4 26.0 mm to (159.1, 53.0), turned to 90 degrees
- moved J6 24.2 mm to (121.2, 71.5)
- moved R2 21.6 mm to (129.6, 62.1), turned to -90 degrees
- moved R3 20.9 mm to (129.2, 82.7), turned to -90 degrees
- moved Q2 19.2 mm to (128.3, 77.2), turned to 180 degrees
- moved D3 19.0 mm to (116.3, 62.0), turned to 180 degrees
- moved D4 18.9 mm to (115.9, 81.7), turned to 180 degrees
- moved J3 18.3 mm to (159.1, 84.6)
- moved Q1 17.4 mm to (128.6, 56.8), turned to 180 degrees
- moved D2 17.2 mm to (129.2, 72.5), turned to -90 degrees
- moved D1 17.0 mm to (129.6, 52.1), turned to -90 degrees
- moved J2 16.2 mm to (159.4, 63.1)
- moved K1 16.2 mm to (133.3, 60.6)
- moved K2 15.5 mm to (133.0, 81.0)
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Connections:
- net /RY-VCC renamed +12V
- net J2 renamed J2-COM
- net J3 renamed J3-COM
- net J4 renamed J4-COM
- net J5 renamed J5-COM
- net Net-(J2-Pin_1) renamed J2-NO
- net Net-(J2-Pin_3) renamed J2-NC
- net Net-(J3-Pin_1) renamed J3-NO
- net Net-(J3-Pin_3) renamed J3-NC
- net Net-(J4-Pin_1) renamed J4-NO
- net Net-(J4-Pin_3) renamed J4-NC
- net Net-(J5-Pin_1) renamed J5-NO
- net Net-(J5-Pin_3) renamed J5-NC
- D3 pad 1: unconnected-(D3-K-Pad1) -> GND
- D4 pad 1: unconnected-(D4-K-Pad1) -> GND
- J1 pad 2: /VCC -> DatIN1
- J6 pad 2: /VCC -> DatIN2
- R1 pad 1: /VCC -> DatIN1
- R4 pad 1: /VCC -> DatIN2
Routing:
- net +12V: track 0.00 -> 239.3 mm, vias 0 -> 5
- net J3-COM: track 0.00 -> 29.8 mm, vias 0 -> 2
- net J2-COM: track 0.00 -> 28.1 mm, vias 0 -> 2
- net J9-COM: track 0.00 -> 26.6 mm, vias 0 -> 2
- net +5V: track 0.00 -> 26.0 mm, vias 0 -> 1
- net J11-COM: track 0.00 -> 25.7 mm, vias 0 -> 1
- net J10-COM: track 0.00 -> 25.2 mm
- net J5-COM: track 0.00 -> 25.1 mm
- net J4-COM: track 0.00 -> 24.0 mm
- net J12-COM: track 0.00 -> 23.9 mm
- net Net-(D1-A): track 0.00 -> 19.0 mm, vias 0 -> 1
- net J4-NC: track 0.00 -> 17.3 mm
- net J10-NC: track 0.00 -> 17.3 mm
- net J5-NC: track 0.00 -> 17.2 mm
- net J12-NC: track 0.00 -> 17.0 mm
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Other:
- board outline removed

Commit message: Terminamos el pcb
Parts:
- removed J1, J6, J7, J8: ~, EESTN5:Jumper
- added SW1: SW_DPST_x2, Button_Switch_THT:SW_PUSH_1P1T_6x3.5mm_H4.3_APEM_MJTP1243, F.Cu at (96.7, 113.1)
- J13: value Screw_Terminal_01x02 -> Screw_Terminal
- R2, R3, R7, R8: value 510 -> 1k
- moved C1 10.2 mm to (91.4, 105.8)
- moved D1 3.53 mm to (126.2, 53.0), turned to 0 degrees
- moved R3 3.34 mm to (126.3, 81.0), turned to 180 degrees
- moved D8 3.32 mm to (126.2, 116.8), turned to 0 degrees
- moved D7 3.17 mm to (126.3, 95.2), turned to 0 degrees
- moved R8 3.11 mm to (126.5, 125.0), turned to 180 degrees
- moved R7 3.04 mm to (126.5, 103.4), turned to 180 degrees
- moved D2 2.96 mm to (126.4, 73.4), turned to 0 degrees
- moved R2 2.88 mm to (126.7, 62.0), turned to 180 degrees
- moved J3 2.80 mm to (161.7, 83.6)
- moved J9 2.70 mm to (161.7, 105.3)
- moved J11 2.69 mm to (161.7, 127.2)
- moved R4 2.66 mm to (113.9, 73.3), turned to 0 degrees
- moved J4 2.65 mm to (161.7, 53.0)
- moved J10 2.59 mm to (161.7, 95.2)
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Connections:
- J13 pad 1: +12V -> Net-(J13-Pin_1)
- U7 pad 21: unconnected-(U7-RX2-Pad21) -> DatIN4
- U7 pad 22: DatIN4 -> DatIN3
- U7 pad 23: DatIN3 -> unconnected-(U7-IO5-Pad23)
Routing:
- net DatIN4: track 3.08 -> 43.5 mm, vias 0 -> 1
- net DatIN3: track 3.14 -> 25.4 mm, vias 0 -> 1
- net DatIN1: track 3.28 -> 20.9 mm, vias 0 -> 1
- net J11-COM: track 25.7 -> 39.0 mm, vias 1 -> 0
- net J9-COM: track 26.6 -> 39.1 mm, vias 2 -> 0
- net Net-(D1-A): track 19.0 -> 9.11 mm
- net J2-COM: track 28.1 -> 37.1 mm, vias 2 -> 0
- net DatIN2: track 3.10 -> 11.1 mm, vias 0 -> 1
- net J3-COM: track 29.8 -> 37.9 mm, vias 2 -> 0
- net Net-(J13-Pin_1): track 0.00 -> 5.93 mm
- net Net-(R3-Pad2): track 10.4 -> 4.95 mm
- net Net-(R8-Pad2): track 10.7 -> 5.30 mm
- net Net-(D2-A): track 13.8 -> 8.52 mm
- net Net-(D8-A): track 14.1 -> 8.89 mm
- net Net-(R7-Pad2): track 10.1 -> 4.99 mm
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- added copper zone on B.Cu, net GND
- added copper zone on F.Cu, net GND

Commit message: Para el Chequeo de Legui
Parts:
- added H1: MountingHole, MountingHole:MountingHole_3.2mm_M3, F.Cu at (76.2, 133.7)
- added H2: MountingHole, MountingHole:MountingHole_3.2mm_M3, F.Cu at (76.3, 43.5)
- added H3: MountingHole, MountingHole:MountingHole_3.2mm_M3, F.Cu at (168.4, 133.8)
- added H4: MountingHole, MountingHole:MountingHole_3.2mm_M3, F.Cu at (168.3, 43.4)
- J13: footprint TerminalBlock:TerminalBlock_bornier-2_P5.08mm -> TerminalBlock:TerminalBlock_MaiXu_MX126-5.0-02P_1x02_P5.00mm
Routing:
- net GND: vias 1 -> 4

Commit message: Ultima Revision
Parts:
- C1, C2, U5: moved to B.Cu
- D1, D2, D7, D8: footprint Diode_SMD:D_0805_2012Metric -> Diode_SMD:D_SMA
- Q1, Q2, Q3, Q4: value ~ -> MMBT2222A
- moved C1 6.40 mm to (91.4, 112.2)
- moved C2 5.36 mm to (81.5, 102.3)
- moved U5 5.10 mm to (83.0, 115.7), turned to 90 degrees
- moved R2 2.98 mm to (123.7, 62.0)
- moved R7 2.86 mm to (123.7, 104.0)
- moved R3 2.77 mm to (123.7, 81.9)
- moved R8 2.76 mm to (123.7, 125.0)
- moved D2 2.07 mm to (125.8, 71.4), turned to -90 degrees
- moved D7 2.06 mm to (125.8, 93.2), turned to -90 degrees
- moved D1 2.02 mm to (125.8, 51.0), turned to -90 degrees
- moved D8 2.01 mm to (126.3, 114.8), turned to -90 degrees
- moved D4 1.62 mm to (115.1, 82.9), turned to 90 degrees
- moved D6 1.52 mm to (115.1, 126.0), turned to 90 degrees
- moved D5 1.48 mm to (115.1, 105.0), turned to 90 degrees
- moved D3 1.37 mm to (115.1, 63.0), turned to 90 degrees
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Connections:
- J10 pad 2: J10-COM -> J10-NC
- J10 pad 3: J10-NC -> J10-COM
- J11 pad 1: J11-NO -> J11-COM
- J11 pad 2: J11-COM -> J11-NO
- J12 pad 2: J12-COM -> J12-NC
- J12 pad 3: J12-NC -> J12-COM
- J2 pad 1: J2-NO -> J2-COM
- J2 pad 2: J2-COM -> J2-NO
- J3 pad 1: J3-NO -> J3-COM
- J3 pad 2: J3-COM -> J3-NO
- J4 pad 2: J4-COM -> J4-NC
- J4 pad 3: J4-NC -> J4-COM
- J5 pad 2: J5-COM -> J5-NC
- J5 pad 3: J5-NC -> J5-COM
- J9 pad 1: J9-NO -> J9-COM
- J9 pad 2: J9-COM -> J9-NO
- Q1 pad 1: GND -> Net-(Q1-B)
- Q1 pad 2: Net-(D1-A) -> GND
- Q1 pad 3: Net-(Q1-B) -> Net-(D1-A)
- Q2 pad 1: GND -> Net-(Q2-B)
- Q2 pad 2: Net-(D2-A) -> GND
- Q2 pad 3: Net-(Q2-B) -> Net-(D2-A)
- Q3 pad 1: GND -> Net-(Q3-B)
- Q3 pad 2: Net-(D7-A) -> GND
- Q3 pad 3: Net-(Q3-B) -> Net-(D7-A)
- Q4 pad 1: GND -> Net-(Q4-B)
- Q4 pad 2: Net-(D8-A) -> GND
- Q4 pad 3: Net-(Q4-B) -> Net-(D8-A)
Routing:
- net +5V: track 23.6 -> 40.7 mm, vias 1 -> 0
- net J9-COM: track 39.1 -> 23.1 mm
- net J11-COM: track 39.0 -> 23.0 mm
- net J3-COM: track 37.9 -> 23.5 mm
- net J2-COM: track 37.1 -> 22.8 mm
- net +12V: track 240.6 -> 229.4 mm, vias 5 -> 4
- net Net-(Q3-B): track 4.09 -> 6.79 mm
- net J4-COM: track 26.9 -> 24.3 mm
- net Net-(D2-A): track 8.52 -> 11.0 mm
- net Net-(R8-Pad2): track 5.30 -> 3.00 mm
- net J9-NO: track 12.9 -> 10.7 mm
- net J4-NC: track 19.6 -> 17.6 mm
- net Net-(R2-Pad2): track 5.83 -> 3.80 mm
- net J3-NO: track 12.9 -> 10.9 mm
- net J5-COM: track 26.9 -> 24.9 mm
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
Commit message: Finalisamos el pcb
Parts:
- added R10: 1k, Resistor_SMD:R_0805_2012Metric_Pad1.20x1.40mm_HandSolder, F.Cu at (128.0, 52.0)
- added R11: 1k, Resistor_SMD:R_0805_2012Metric_Pad1.20x1.40mm_HandSolder, F.Cu at (128.0, 94.2)
- added R12: 1k, Resistor_SMD:R_0805_2012Metric_Pad1.20x1.40mm_HandSolder, F.Cu at (128.0, 115.8)
- added R9: 1k, Resistor_SMD:R_0805_2012Metric_Pad1.20x1.40mm_HandSolder, F.Cu at (128.0, 72.4)
- R1, R4, R5, R6: value 1K -> 100
- moved D3 14.8 mm to (123.7, 51.0), turned to 180 degrees
- moved D5 14.7 mm to (123.7, 93.2), turned to 180 degrees
- moved D4 14.4 mm to (123.7, 71.4), turned to 180 degrees
- moved D6 14.2 mm to (123.7, 114.8), turned to 180 degrees
- moved D1 5.46 mm to (131.3, 51.0)
- moved D2 5.46 mm to (131.3, 71.4)
- moved D7 5.46 mm to (131.3, 93.2)
- moved D8 5.01 mm to (131.3, 114.8)
- moved K2 4.42 mm to (137.4, 81.0)
- moved K4 4.29 mm to (137.4, 124.4)
- moved K3 4.24 mm to (137.4, 102.8)
- moved K1 4.07 mm to (137.4, 60.6)
- moved R4 1.88 mm to (114.1, 71.4)
- moved Q1 1.50 mm to (128.0, 56.9)
- moved Q3 1.43 mm to (128.0, 99.1)
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Connections:
- D3 pad 1: GND -> Net-(D3-K)
- D3 pad 2: Net-(D3-A) -> +12V
- D4 pad 1: GND -> Net-(D4-K)
- D4 pad 2: Net-(D4-A) -> +12V
- D5 pad 1: GND -> Net-(D5-K)
- D5 pad 2: Net-(D5-A) -> +12V
- D6 pad 1: GND -> Net-(D6-K)
- D6 pad 2: Net-(D6-A) -> +12V
- U1 pad 2: Net-(D4-A) -> GND
- U2 pad 2: Net-(D3-A) -> GND
- U3 pad 2: Net-(D5-A) -> GND
- U4 pad 2: Net-(D6-A) -> GND
Routing:
- net +12V: track 229.4 -> 251.0 mm
- net J3-COM: track 23.5 -> 18.5 mm
- net J5-NC: track 18.2 -> 13.5 mm
- net J10-COM: track 25.1 -> 20.5 mm
- net J9-COM: track 23.1 -> 18.5 mm
- net J5-NO: track 10.9 -> 6.50 mm
- net J3-NO: track 10.9 -> 6.50 mm
- net J11-NO: track 10.9 -> 6.50 mm
- net J10-NC: track 17.8 -> 13.5 mm
- net J11-NC: track 17.6 -> 13.3 mm
- net J12-NC: track 17.8 -> 13.5 mm
- net J12-COM: track 25.1 -> 20.8 mm
- net J9-NC: track 17.8 -> 13.5 mm
- net J11-COM: track 23.0 -> 18.7 mm
- net J3-NC: track 17.9 -> 13.6 mm
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
Commit message: Ya esta para imprimir
Parts:
- removed H4: MountingHole, MountingHole:MountingHole_3.2mm_M3
- added G***: LOGO, EESTN5:Caballerito, F.Cu at (87.3, 115.6)
- added G***: LOGO, EESTN5:Caballerito, B.Cu at (87.3, 115.6)
- added J1: ULTRASONIDO, Connector_PinHeader_2.54mm:PinHeader_1x04_P2.54mm_Vertical, B.Cu at (86.7, 71.7)
- added R13: 1k, Resistor_THT:R_Axial_DIN0204_L3.6mm_D1.6mm_P7.62mm_Horizontal, B.Cu at (91.1, 69.2)
- added R14: 1k, Resistor_THT:R_Axial_DIN0204_L3.6mm_D1.6mm_P7.62mm_Horizontal, B.Cu at (98.8, 74.5)
- moved U5 24.8 mm to (93.2, 93.0)
- moved C1 15.6 mm to (102.0, 100.7), turned to 0 degrees
- moved H3 7.47 mm to (162.4, 129.3)
- moved H2 7.14 mm to (81.3, 48.6)
- moved H1 6.77 mm to (81.3, 129.3)
- moved J13 6.22 mm to (101.0, 121.1)
- moved SW1 6.14 mm to (101.0, 108.8)
- moved J11 3.36 mm to (161.7, 123.6)
- moved K4 3.36 mm to (137.4, 121.1)
- moved Q4 3.36 mm to (127.9, 117.3)
- moved R8 3.36 mm to (123.7, 121.6)
- moved U4 3.36 mm to (115.1, 116.1)
- moved D6 3.36 mm to (123.7, 111.5)
- moved D8 3.36 mm to (131.3, 111.5)
- moved J12 3.36 mm to (161.7, 113.5)
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Connections:
- U7 pad 4: unconnected-(U7-IO34-Pad4) -> D Echo
- U7 pad 6: unconnected-(U7-IO32-Pad6) -> Trig
Routing:
- net D Echo: track 0.00 -> 29.4 mm
- net +12V: track 251.0 -> 228.9 mm
- net Trig: track 0.00 -> 6.15 mm
- net Echo: track 0.00 -> 4.49 mm
- net DatIN4: track 43.9 -> 40.7 mm
- net +5V: track 40.7 -> 43.1 mm
- net DatIN3: track 25.3 -> 23.4 mm
- net GND: vias 1 -> 0
Other:
- board text added: "Agustin Mayans 6°5°"

Commit message: A imprimir
Parts:
- added C1: 0.33 uF, Capacitor_SMD:C_0805_2012Metric, F.Cu at (249.3, 100.7)
- added C2: 0.1 uF, Capacitor_SMD:C_0805_2012Metric, F.Cu at (271.8, 100.7)
- added D1: ~, Diode_SMD:D_SMA, B.Cu at (220.0, 51.0)
- added D2: ~, Diode_SMD:D_SMA, B.Cu at (220.0, 71.2)
- added D3: ~, EESTN5:Led_0805, B.Cu at (227.6, 51.0)
- added D4: ~, EESTN5:Led_0805, B.Cu at (227.6, 71.2)
- added D5: ~, EESTN5:Led_0805, B.Cu at (227.6, 91.3)
- added D6: ~, EESTN5:Led_0805, B.Cu at (227.6, 111.5)
- added D7: ~, Diode_SMD:D_SMA, B.Cu at (220.0, 91.3)
- added D8: ~, Diode_SMD:D_SMA, B.Cu at (220.0, 111.5)
- added G***: LOGO, EESTN5:Caballerito, F.Cu at (264.0, 115.6)
- added G***: LOGO, EESTN5:Caballerito, B.Cu at (264.0, 115.6)
- added H1: MountingHole, MountingHole:MountingHole_3.2mm_M3, B.Cu at (270.0, 129.3)
- added H2: MountingHole, MountingHole:MountingHole_3.2mm_M3, B.Cu at (270.0, 48.6)
- added H3: MountingHole, MountingHole:MountingHole_3.2mm_M3, B.Cu at (188.9, 129.3)
- added J1: ULTRASONIDO, Connector_PinHeader_2.54mm:PinHeader_1x04_P2.54mm_Vertical, F.Cu at (264.7, 71.7)
- added J10: ~, TerminalBlock:TerminalBlock_Xinya_XY308-2.54-3P_1x03_P2.54mm_Horizontal, B.Cu at (189.6, 93.3)
- added J11: ~, TerminalBlock:TerminalBlock_Xinya_XY308-2.54-3P_1x03_P2.54mm_Horizontal, B.Cu at (189.6, 123.6)
- added J12: ~, TerminalBlock:TerminalBlock_Xinya_XY308-2.54-3P_1x03_P2.54mm_Horizontal, B.Cu at (189.6, 113.5)
- added J13: Screw_Terminal, TerminalBlock:TerminalBlock_MaiXu_MX126-5.0-02P_1x02_P5.00mm, B.Cu at (250.3, 121.1)
- added J2: ~, TerminalBlock:TerminalBlock_Xinya_XY308-2.54-3P_1x03_P2.54mm_Horizontal, B.Cu at (189.6, 63.2)
- added J3: ~, TerminalBlock:TerminalBlock_Xinya_XY308-2.54-3P_1x03_P2.54mm_Horizontal, B.Cu at (189.6, 83.3)
- added J4: ~, TerminalBlock:TerminalBlock_Xinya_XY308-2.54-3P_1x03_P2.54mm_Horizontal, B.Cu at (189.6, 53.0)
- added J5: ~, TerminalBlock:TerminalBlock_Xinya_XY308-2.54-3P_1x03_P2.54mm_Horizontal, B.Cu at (189.6, 73.2)
- added J9: ~, TerminalBlock:TerminalBlock_Xinya_XY308-2.54-3P_1x03_P2.54mm_Horizontal, B.Cu at (189.6, 103.4)
- added K1: ~, Relay_THT:Relay_DPDT_Finder_30.22, B.Cu at (213.9, 60.6)
- added K2: ~, Relay_THT:Relay_DPDT_Finder_30.22, B.Cu at (213.9, 80.8)
- added K3: ~, Relay_THT:Relay_DPDT_Finder_30.22, B.Cu at (213.9, 100.9)
- added K4: ~, Relay_THT:Relay_DPDT_Finder_30.22, B.Cu at (213.9, 121.1)
- added Q1: MMBT2222A, Package_TO_SOT_SMD:SOT-23, B.Cu at (223.4, 56.9)
- added Q2: MMBT2222A, Package_TO_SOT_SMD:SOT-23, B.Cu at (223.4, 77.9)
- added Q3: MMBT2222A, Package_TO_SOT_SMD:SOT-23, B.Cu at (223.4, 97.2)
- added Q4: MMBT2222A, Package_TO_SOT_SMD:SOT-23, B.Cu at (223.4, 117.3)
- added R1: 100, Resistor_SMD:R_0805_2012Metric_Pad1.20x1.40mm_HandSolder, B.Cu at (237.2, 51.0)
- added R10: 1k, Resistor_SMD:R_0805_2012Metric_Pad1.20x1.40mm_HandSolder, B.Cu at (223.4, 52.0)
- added R11: 1k, Resistor_SMD:R_0805_2012Metric_Pad1.20x1.40mm_HandSolder, B.Cu at (223.4, 92.3)
- added R12: 1k, Resistor_SMD:R_0805_2012Metric_Pad1.20x1.40mm_HandSolder, B.Cu at (223.4, 112.5)
- added R13: 1k, Resistor_SMD:R_0805_2012Metric_Pad1.20x1.40mm_HandSolder, F.Cu at (258.5, 69.2)
- added R14: 2k, Resistor_SMD:R_0805_2012Metric_Pad1.20x1.40mm_HandSolder, F.Cu at (252.9, 69.2)
- added R2: 1k, Resistor_SMD:R_0805_2012Metric_Pad1.20x1.40mm_HandSolder, B.Cu at (227.6, 62.0)
- added R3: 1k, Resistor_SMD:R_0805_2012Metric_Pad1.20x1.40mm_HandSolder, B.Cu at (227.6, 81.7)
- added R4: 100, Resistor_SMD:R_0805_2012Metric_Pad1.20x1.40mm_HandSolder, B.Cu at (237.2, 71.2)
- added R5: 100, Resistor_SMD:R_0805_2012Metric_Pad1.20x1.40mm_HandSolder, B.Cu at (237.3, 91.3)
- added R6: 100, Resistor_SMD:R_0805_2012Metric_Pad1.20x1.40mm_HandSolder, B.Cu at (237.3, 111.5)
- added R7: 1k, Resistor_SMD:R_0805_2012Metric_Pad1.20x1.40mm_HandSolder, B.Cu at (227.6, 102.1)
- added R8: 1k, Resistor_SMD:R_0805_2012Metric_Pad1.20x1.40mm_HandSolder, B.Cu at (227.6, 121.6)
- added R9: 1k, Resistor_SMD:R_0805_2012Metric_Pad1.20x1.40mm_HandSolder, B.Cu at (223.4, 72.2)
- added SW1: SW_DPST_x2, Button_Switch_THT:SW_PUSH_1P1T_6x3.5mm_H4.3_APEM_MJTP1243, B.Cu at (250.3, 108.8)
- added U1: 817C, Package_DIP:DIP-4_W7.62mm, B.Cu at (236.2, 75.8)
- added U2: 817C, Package_DIP:DIP-4_W7.62mm, B.Cu at (236.2, 55.6)
- added U3: 817C, Package_DIP:DIP-4_W7.62mm, B.Cu at (236.3, 96.3)
- added U4: 817C, Package_DIP:DIP-4_W7.62mm, B.Cu at (236.3, 116.1)
- added U5: L7805, Package_TO_SOT_SMD:TO-263-3_TabPin2, F.Cu at (258.1, 93.0)
- added U7: ESP32_DevKit_V1_CH9102X, EESTN5:ESP32-WROOM-32.30pines, B.Cu at (257.5, 68.0)
- R13: footprint Resistor_THT:R_Axial_DIN0204_L3.6mm_D1.6mm_P7.62mm_Horizontal -> Resistor_SMD:R_0805_2012Metric_Pad1.20x1.40mm_HandSolder
- R14: value 1k -> 2k; footprint Resistor_THT:R_Axial_DIN0204_L3.6mm_D1.6mm_P7.62mm_Horizontal -> Resistor_SMD:R_0805_2012Metric_Pad1.20x1.40mm_HandSolder
- moved R14 5.40 mm to (98.4, 69.2), turned to 0 degrees
- moved R13 1.66 mm to (92.8, 69.2)
Routing:
- net +12V: track 228.9 -> 457.7 mm, vias 4 -> 8
- net +5V: track 43.1 -> 86.1 mm
- net DatIN4: track 40.7 -> 81.4 mm, vias 1 -> 2
- net DatIN3: track 23.4 -> 46.9 mm, vias 1 -> 2
- net D Echo: track 29.4 -> 52.2 mm
- net DatIN1: track 21.8 -> 43.5 mm, vias 1 -> 2
- net J12-COM: track 20.8 -> 41.5 mm
- net J4-COM: track 20.8 -> 41.5 mm
- net J5-COM: track 20.6 -> 41.2 mm
- net J10-COM: track 20.5 -> 41.1 mm
- net J11-COM: track 18.7 -> 37.4 mm
- net J2-COM: track 18.6 -> 37.3 mm
- net J9-COM: track 18.5 -> 37.1 mm
- net J3-COM: track 18.5 -> 37.0 mm
- net J3-NC: track 13.6 -> 27.2 mm
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Other:
- board text added: "Mayans / Zacarias 6°5°"
- board text removed: "Agustin Mayans 6°5°"
